File: L240-1.brd (EAGLE design)
At the start: 160 x 100 mm, 13 parts, among them IC1 TINY13-20SSU, IC2 LM1117IMPX-3.3, X2 22-23-2021, X3 MKDSN1,5/6-5,08

Commit message: relay
Parts:
- removed D9: DIODE1N4007, MyLib:SMA-DIODE
- added D1: DIODE1N4007, MyLib:SMA-DIODE
- added K1: G6RW, relay:G6RW
- added X1: MKDSN1,5/2-5,08, con-phoenix-508:MKDSN1,5/2-5,08
- X3: value MKDSN1,5/6-5,08 -> MKDSN1,5/2-5,08; device con-phoenix-508:MKDSN1,5/6-5,08 -> con-phoenix-508:MKDSN1,5/2-5,08
- moved X3 18.8 mm to (81.7, 46.5), turned to 270 degrees
- moved Q3 11.7 mm to (64.9, 32.7)
- moved R6 7.69 mm to (59.9, 33.6)
Connections:
- removed net GND1: Q3.2
- new net N$1: X1.1, X3.2
- new net N$2: K1.S, X3.1
- new net N$3: K1.P, X1.2
- net +5V: now also D1.C, K1.2; no longer D9.C
- net GND: now also Q3.2
- net N$13: now also D1.A, K1.1; no longer D9.A, X3.5
Changed lines of the file:
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@@
 </autorouter>
 <elements>
-<element name="D9" library="MyLib" package="SMA-DIODE" value="DIODE1N4007" x="81.28" y="40.64" smashed="yes" rot="R90">
-<attribute name="NAME" x="79.629" y="40.64" size="0.6096" layer="25" font="vector" ratio="20" rot="R90" align="bottom-center"/>
-<attribute name="VALUE" x="82.931" y="40.64" size="0.6096" layer="27" font="vector" ratio="20" rot="R90" align="top-center"/>
-</element>
 <element name="IC1" library="atmel" library_urn="urn:adsk.eagle:library:105" package="8S1" package3d_urn="urn:adsk.eagle:package:4358/1" value="TINY13-20SSU" x="52.07" y="33.02" smashed="yes">
 <attribute name="MF" value="" x="69.85" y="29.21" size="1.778" layer="27" display="off"/>
@@
 <attribute name="VALUE" x="56.134" y="30.861" size="1.27" layer="27" ratio="10" rot="R90"/>
 </element>
-<element name="Q3" library="MyLib" package="SOT23-WIDE" value="" x="75.184" y="38.227" smashed="yes" rot="R270">
-<attribute name="NAME" x="75.184" y="36.322" size="0.8128" layer="25" ratio="18" rot="R270"/>
-<attribute name="VALUE" x="74.549" y="36.322" size="0.4064" layer="27" ratio="10" rot="R270"/>
+<element name="Q3" library="MyLib" package="SOT23-WIDE" value="" x="64.904934375" y="32.659959375" smashed="yes" rot="R270">
+<attribute name="NAME" x="64.904934375" y="30.754959375" size="0.8128" layer="25" ratio="18" rot="R270"/>
+<attribute name="VALUE" x="64.269934375" y="30.754959375" size="0.4064" layer="27" ratio="10" rot="R270"/>
 </element>
-<element name="R6" library="rcl" package="R0805" value="50" x="67.31" y="35.56" smashed="yes" rot="R180">
-<attribute name="NAME" x="67.945" y="34.29" size="1.27" layer="25" rot="R180"/>
-<attribute name="VALUE" x="67.945" y="38.1" size="1.27" layer="27" rot="R180"/>
-</element>
-<element name="X3" library="con-phoenix-508" library_urn="urn:adsk.eagle:library:176" package="MKDSN1,5/6-5,08" package3d_urn="urn:adsk.eagle:package:9634/1" value="MKDSN1,5/6-5,08" x="91.44" y="30.48" smashed="yes" rot="R90">
-<attribute name="NAME" x="86.995" y="15.59" size="1.27" layer="25" rot="R90"/>
-<attribute name="POPULARITY" value="0" x="110.49" y="59.69" size="1.778" layer="27" rot="R90" display="off"/>
-<attribute name="VALUE" x="86.995" y="24.13" size="1.27" layer="27" rot="R90"/>
+<element name="R6" library="rcl" package="R0805" value="50" x="59.882084375" y="33.567371875" smashed="yes" rot="R180">
+<attribute name="NAME" x="60.517084375" y="32.297371875" size="1.27" layer="25" rot="R180"/>
+<attribute name="VALUE" x="60.517084375" y="36.107371875" size="1.27" layer="27" rot="R180"/>
 </element>
 <element name="C13" library="rcl" package="C0805" value="0.1" x="22.183090625" y="32.276415625" smashed="yes" rot="R180">
@@
 <attribute name="VALUE" x="54.022625" y="36.917625" size="1.27" layer="28" rot="MR0"/>
 </element>
+<element name="X1" library="con-phoenix-508" library_urn="urn:adsk.eagle:library:176" package="MKDSN1,5/2-5,08" package3d_urn="urn:adsk.eagle:package:9630/1" value="MKDSN1,5/2-5,08" x="81.6413125" y="27.93968125" smashed="yes" rot="R270">
+<attribute name="NAME" x="86.0863125" y="32.69078125" size="1.27" layer="25" rot="R270"/>
+<attribute name="POPULARITY" value="14" x="81.6413125" y="27.93968125" size="1.778" layer="27" rot="R270" display="off"/>
+<attribute name="VALUE" x="77.8313125" y="20.95468125" size="1.27" layer="27"/>
+</element>
+<element name="K1" library="relay" library_urn="urn:adsk.eagle:library:339" package="G6RW" package3d_urn="urn:adsk.eagle:package:24332/1" value="G6RW" x="67.954521875" y="36.600446875" smashed="yes" rot="MR90">
+<attribute name="MF" value="" x="67.954521875" y="36.600446875" size="1.778" layer="28" rot="MR90" display="off"/>
+<attribute name="MPN" value="" x="67.954521875" y="36.600446875" size="1.778" layer="28" rot="MR90" display="off"/>
+<attribute name="NAME" x="62.874521875" y="53.110446875" size="1.778" layer="26" ratio="10" rot="MR180"/>
+<attribute name="OC_FARNELL" value="unknown" x="67.954521875" y="36.600446875" size="1.778" layer="28" rot="MR90" display="off"/>
+<attribute name="OC_NEWARK" value="unknown" x="67.954521875" y="36.600446875" size="1.778" layer="28" rot="MR90" display="off"/>
+<attribute name="POPULARITY" value="1" x="67.954521875" y="36.600446875" size="1.778" layer="28" rot="MR90" display="off"/>
+<attribute name="VALUE" x="67.065521875" y="28.980446875" size="1.778" layer="28" ratio="10" rot="MR90"/>
+</element>
+<element name="X3" library="con-phoenix-508" library_urn="urn:adsk.eagle:library:176" package="MKDSN1,5/2-5,08" package3d_urn="urn:adsk.eagle:package:9630/1" value="MKDSN1,5/2-5,08" x="81.723546875" y="46.52930625" smashed="yes" rot="R270">
+<attribute name="NAME" x="86.168546875" y="51.28040625" size="1.27" layer="25" rot="R270"/>
+<attribute name="POPULARITY" value="14" x="86.835615625" y="46.52930625" size="1.778" layer="27" rot="R270" display="off"/>
+<attribute name="VALUE" x="77.913546875" y="39.54430625" size="1.27" layer="27"/>
+</element>
+<element name="D1" library="MyLib" package="SMA-DIODE" value="DIODE1N4007" x="68.1583625" y="28.570553125" smashed="yes">
+<attribute name="NAME" x="68.1583625" y="30.221553125" size="0.6096" layer="25" font="vector" ratio="20" align="bottom-center"/>
+<attribute name="VALUE" x="68.1583625" y="26.919553125" size="0.6096" layer="27" font="vector" ratio="20" align="top-center"/>
+</element>
 </elements>
 <signals>
@@
 <contactref element="JP1" pad="6"/>
 <contactref element="IC1" pad="4"/>
-<wire x1="53.965" y1="30.366" x2="47.672625" y2="42.632625" width="0" layer="19" extent="1-1"/>
+<contactref element="Q3" pad="2"/>
+<wire x1="53.965" y1="30.366" x2="63.904934375" y2="31.709959375" width="0" layer="19" extent="1-1"/>
 <wire x1="46.200059375" y1="32.021421875" x2="53.965" y2="30.366" width="0" layer="19" extent="1-1"/>
-<wire x1="29.83420625" y1="40.41296875" x2="46.200059375" y2="32.021421875" width="0" layer="19" extent="1-1"/>
+<wire x1="47.672625" y1="42.632625" x2="46.200059375" y2="32.021421875" width="0" layer="19" extent="1-1"/>
+<wire x1="29.83420625" y1="40.41296875" x2="47.672625" y2="42.632625" width="0" layer="19" extent="1-1"/>
 <wire x1="23.312321875" y1="35.737246875" x2="29.83420625" y2="40.41296875" width="0" layer="19" extent="1-1"/>
 <wire x1="21.233090625" y1="32.276415625" x2="23.312321875" y2="35.737246875" width="0" layer="19" extent="1-1"/>
@@
 <contactref element="R6" pad="2"/>
 <contactref element="IC1" pad="3"/>
-<wire x1="52.695" y1="30.366" x2="66.36" y2="35.56" width="0" layer="19" extent="1-1"/>
+<wire x1="52.695" y1="30.366" x2="58.932084375" y2="33.567371875" width="0" layer="19" extent="1-1"/>
 </signal>
 <signal name="N$11">
 <contactref element="Q3" pad="1"/>
 <contactref element="R6" pad="1"/>
-<wire x1="68.26" y1="35.56" x2="74.184" y2="39.177" width="0" layer="19" extent="1-1"/>
+<wire x1="60.832084375" y1="33.567371875" x2="63.904934375" y2="33.609959375" width="0" layer="19" extent="1-1"/>
 </signal>
 <signal name="N$13">
-<contactref element="D9" pad="A"/>
 <contactref element="Q3" pad="3"/>
-<contactref element="X3" pad="5"/>
-<wire x1="81.28" y1="38.49" x2="91.415" y2="38.1" width="0" layer="19" extent="1-1"/>
-<wire x1="76.184" y1="38.227" x2="81.28" y2="38.49" width="0" layer="19" extent="1-1"/>
-</signal>
-<signal name="GND1">
-<contactref element="Q3" pad="2"/>
+<contactref element="D1" pad="A"/>
+<contactref element="K1" pad="1"/>
+<wire x1="66.0083625" y1="28.570553125" x2="65.904934375" y2="32.659959375" width="0" layer="19" extent="1-1"/>
+<wire x1="64.144521875" y1="23.900446875" x2="66.0083625" y2="28.570553125" width="0" layer="19" extent="1-1"/>
 </signal>
 <signal name="+3V3">
@@
 <contactref element="C10" pad="1"/>
 <contactref element="C6" pad="+"/>
-<contactref element="D9" pad="C"/>
-<wire x1="23.256590625" y1="43.759434375" x2="81.28" y2="42.79" width="0" layer="19" extent="1-1"/>
-<wire x1="23.312321875" y1="40.359246875" x2="23.256590625" y2="43.759434375" width="0" layer="19" extent="1-1"/>
+<contactref element="K1" pad="2"/>
+<contactref element="D1" pad="C"/>
+<wire x1="71.764521875" y1="23.900446875" x2="70.3083625" y2="28.570553125" width="0" layer="19" extent="1-1"/>
+<wire x1="23.312321875" y1="40.359246875" x2="70.3083625" y2="28.570553125" width="0" layer="19" extent="1-1"/>
+<wire x1="23.256590625" y1="43.759434375" x2="23.312321875" y2="40.359246875" width="0" layer="19" extent="1-1"/>
 <wire x1="10.699434375" y1="41.145759375" x2="23.312321875" y2="40.359246875" width="0" layer="19" extent="1-1"/>
 <wire x1="2.530790625" y1="40.125015625" x2="10.699434375" y2="41.145759375" width="0" layer="19" extent="1-1"/>
@@
 <wire x1="50.165" y1="30.366" x2="47.672625" y2="40.092625" width="0" layer="19" extent="1-1"/>
 </signal>
+<signal name="N$1">
+<contactref element="X1" pad="1"/>
+<contactref element="X3" pad="2"/>
+<wire x1="81.6663125" y1="30.50078125" x2="81.748546875" y2="44.01040625" width="0" layer="19" extent="1-1"/>
+</signal>
+<signal name="N$2">
+<contactref element="X3" pad="1"/>
+<contactref element="K1" pad="S"/>
+<wire x1="71.764521875" y1="49.300446875" x2="81.748546875" y2="49.09040625" width="0" layer="19" extent="1-1"/>
+</signal>
+<signal name="N$3">
+<contactref element="K1" pad="P"/>
+<contactref element="X1" pad="2"/>
+<wire x1="81.6663125" y1="25.42078125" x2="64.144521875" y2="46.125446875" width="0" layer="19" extent="1-1"/>
+</signal>
 </signals>

Commit message: wip
Parts:
- removed X1, X3: MKDSN1,5/2-5,08, con-phoenix-508:MKDSN1,5/2-5,08
- added C1, C3, C4: 0.1, rcl:C0805
- added C2: 1nF, rcl:C0805
- added IC3: ACS712-LC, allegro-2:SOIC8
- added U$1: KQ130, MyLib:KQ130
- added X4: MKDSN1,5/4-5,08, con-phoenix-508:MKDSN1,5/4-5,08
- K1: value G6RW -> G2R2; device relay:G6RW -> relay:G2R2
- moved C13 115.9 mm to (135.4, 56.8), turned to 270 degrees
- moved C15 103.5 mm to (131.5, 56.8), turned to 90 degrees
- moved C6 101.4 mm to (110.2, 57.8)
- moved IC2 101.4 mm to (119.8, 57.4)
- moved X2 101.4 mm to (102.1, 58.2)
- moved C10 91.8 mm to (113.0, 57.6), turned to 270 degrees
- moved C14 83.7 mm to (126.6, 56.2)
- moved K1 27.5 mm to (41.4, 43.5), turned to 0 degrees
- moved Q3 25.9 mm to (39.9, 39.3)
- moved R6 24.4 mm to (38.8, 45.8), turned to 90 degrees
- moved D1 23.4 mm to (50.2, 43.5), turned to 90 degrees
- moved IC1 10.8 mm to (41.5, 30.8), turned to 180 degrees
- moved JP1 10.5 mm to (51.9, 30.9), turned to 90 degrees
Connections:
- new net LOAD: IC1.2, IC3.7
- new net N$4: IC3.3, IC3.4, X4.1
- new net N$6: K1.S2, X4.2
- new net N$7: C2.1, IC3.6
- net +3V3: no longer IC1.8, JP1.2
- net +5V: now also C1.1, C3.1, C4.1, IC1.8, IC3.8, JP1.2; no longer IC2.3
- net GND: now also C1.2, C2.2, C3.2, C4.2, IC3.5
- net N$1: now also K1.S1, X4.3; no longer X1.1, X3.2
- net N$2: now also IC3.1, IC3.2, K1.P2; no longer K1.S, X3.1
- net N$3: now also K1.P1, X4.4; no longer K1.P, X1.2
Routing:
- net +5V: track 0.00 -> 45.5 mm
- net LOAD: track 0.00 -> 30.0 mm
- net SCK: track 0.00 -> 22.1 mm
- net MOSI: track 0.00 -> 16.5 mm
- net MISO: track 0.00 -> 11.6 mm
- net RESET: track 0.00 -> 7.27 mm

Commit message: v0.1
Parts:
- removed C13, C14: 0.1, rcl:C0805
- removed C15: (no value), rcl:153CLV-0605
- removed IC2: LM1117IMPX-3.3, lm1117:SOT223
- removed JP1: (no value), pinhead:2X03
- removed U$1: KQ130, MyLib:KQ130
- removed X2: 22-23-2021, con-molex:22-23-2021
- added HLK1: HLK-PM013W, hi-link:HLK-PM01
- added MD1: KQ130, MyLib:KQ130
- moved C10 65.4 mm to (47.7, 54.9)
- moved C6 55.1 mm to (55.3, 54.6)
- moved C3 35.5 mm to (31.1, 54.8), turned to 270 degrees
- moved IC1 24.8 mm to (36.0, 54.9), turned to 0 degrees
- moved C4 13.6 mm to (51.9, 34.0), turned to 270 degrees
- moved IC3 10.1 mm to (21.9, 23.6)
- moved C2 9.81 mm to (20.0, 16.3), turned to 90 degrees
- moved D1 9.78 mm to (48.3, 33.9)
- moved C1 9.48 mm to (27.1, 20.1), turned to 270 degrees
- moved K1 9.40 mm to (41.4, 34.1)
- moved R6 8.84 mm to (39.4, 37.0)
- moved Q3 8.84 mm to (40.4, 30.5)
- moved X4 7.18 mm to (5.75, 33.9)
Connections:
- net N$1 renamed N-OUT
- net N$6 renamed L-OUT
- removed net +3V3: C13.1, C14.1, C15.+, IC2.2, IC2.TAB
- removed net N$3: K1.P1, X4.4
- removed net N$4: IC3.3, IC3.4, X4.1
- new net L-IN: HLK1.P$2, IC3.3, IC3.4, MD1.AC2, X4.1
- new net N-IN: HLK1.P$1, K1.P1, MD1.AC1, X4.4
- net +5V: now also HLK1.P$4, MD1.VCC@1, MD1.VCC@2; no longer JP1.2, X2.1
- net GND: now also HLK1.P$3, MD1.GND; no longer C13.2, C14.2, C15.-, IC2.1, JP1.6, X2.2
- net MISO: now also MD1.TX; no longer JP1.1
- net MOSI: now also MD1.RX; no longer JP1.4
- net RESET: no longer JP1.5
- net SCK: no longer JP1.3
Routing:
- net +5V: track 45.5 -> 211.8 mm
- net N-IN: track 0.00 -> 69.8 mm, vias 0 -> 1
- net L-IN: track 0.00 -> 50.1 mm
- net MISO: track 11.6 -> 41.8 mm
- net GND: track 0.00 -> 22.8 mm
- net SCK: track 22.1 -> 0.00 mm
- net MOSI: track 16.5 -> 37.2 mm
- net LOAD: track 30.0 -> 14.7 mm
- net N-OUT: track 0.00 -> 14.9 mm
- net L-OUT: track 0.00 -> 14.0 mm
- net N$13: track 0.00 -> 8.24 mm
- net N$7: track 0.00 -> 7.64 mm
- net RESET: track 7.27 -> 0.00 mm
- net N$2: track 0.00 -> 5.60 mm
- net N$11: track 0.00 -> 4.62 mm
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
Commit message: v0.2
Parts:
- moved X4 101.5 mm to (101.9, 66.6), turned to 270 degrees
- moved C2 95.7 mm to (87.6, 84.1), turned to 270 degrees
- moved IC3 83.1 mm to (85.7, 76.8), turned to 0 degrees
- moved C1 76.5 mm to (76.7, 78.4)
- moved C4 43.1 mm to (67.8, 74.1), turned to 90 degrees
- moved Q3 42.4 mm to (68.8, 61.9), turned to 90 degrees
- moved K1 40.7 mm to (66.3, 66.3), turned to 180 degrees
- moved D1 39.1 mm to (67.8, 67.9)
- moved R6 35.8 mm to (68.6, 57.7), turned to 180 degrees
- moved IC1 24.8 mm to (47.3, 77.0), turned to 180 degrees
- moved C3 22.5 mm to (38.6, 76.0), turned to 0 degrees
Connections:
- net +5V: now also K1.1; no longer K1.2
- net N$13: now also K1.2; no longer K1.1
Routing:
- net L-IN: track 50.1 -> 173.3 mm
- net N-IN: track 69.8 -> 175.3 mm
- net +5V: track 211.8 -> 130.0 mm
- net MISO: track 41.8 -> 4.87 mm
- net LOAD: track 14.7 -> 51.3 mm
- net MOSI: track 37.2 -> 4.36 mm
- net N$13: track 8.24 -> 0.00 mm
- net N$11: track 4.62 -> 0.00 mm
- net OUT1: track 2.78 -> 0.00 mm

Commit message: v0.3
Parts:
- moved Q3 25.3 mm to (47.9, 47.7), turned to 270 degrees
- moved R6 22.1 mm to (46.9, 53.4), turned to 90 degrees
- moved D1 18.7 mm to (54.0, 55.2)
- moved C4 18.4 mm to (54.1, 61.9)
- moved X4 17.9 mm to (88.0, 55.2)
- moved K1 17.4 mm to (52.6, 55.5)
- moved IC3 16.7 mm to (71.9, 67.6)
- moved C2 16.1 mm to (73.5, 76.4), turned to 0 degrees
- moved HLK1 14.2 mm to (18.8, 54.5)
- moved C10 14.1 mm to (33.6, 55.5)
- moved C6 14.0 mm to (41.2, 54.8)
- moved C3 7.77 mm to (33.7, 70.0), turned to 180 degrees
- moved C1 5.72 mm to (78.0, 72.9), turned to 180 degrees
Connections:
- net LOAD: now also IC1.3; no longer IC1.2
- net OUT1: now also IC1.2; no longer IC1.3
Routing:
- net OUT1: track 0.00 -> 58.9 mm
- net +5V: track 130.0 -> 75.4 mm
- net N-IN: track 175.3 -> 151.5 mm, vias 1 -> 0
- net L-IN: track 173.3 -> 159.5 mm
- net LOAD: track 51.3 -> 40.4 mm
- net N$13: track 0.00 -> 10.5 mm
- net N$7: track 7.64 -> 0.00 mm
- net N$11: track 0.00 -> 3.79 mm
- net GND: track 22.8 -> 20.8 mm
- net N$2: track 5.60 -> 7.20 mm
- net N-OUT: track 14.9 -> 14.2 mm

Commit message: v0.4
Parts:
- added JP1: (no value), pinhead:1X06
- moved IC1 44.6 mm to (66.7, 36.7), turned to 90 degrees
- moved C1 44.3 mm to (67.6, 29.8)
- moved IC3 37.7 mm to (75.5, 30.0)
- moved D1 37.5 mm to (53.9, 17.7)
- moved Q3 37.5 mm to (47.8, 10.2)
- moved R6 37.5 mm to (46.8, 15.9)
- moved X4 37.5 mm to (87.9, 17.7)
- moved K1 37.5 mm to (52.5, 17.9)
- moved C10 37.0 mm to (32.8, 18.5)
- moved C3 37.0 mm to (32.9, 33.0)
- moved C6 37.0 mm to (40.5, 17.9)
- moved MD1 37.0 mm to (21.8, 33.0)
- moved HLK1 37.0 mm to (18.0, 17.5)
- moved C2 36.9 mm to (76.2, 39.6), turned to 90 degrees
- moved C4 34.3 mm to (54.4, 27.6), turned to 0 degrees
Connections:
- net +5V: now also JP1.1
- net GND: now also JP1.6
- net MISO: now also JP1.3
- net MOSI: now also JP1.4
- net RESET: now also JP1.5
- net SCK: now also JP1.2
Routing:
- net LOAD: track 40.4 -> 9.04 mm
- net +5V: track 75.4 -> 100.4 mm
- net OUT1: track 58.9 -> 41.3 mm, vias 0 -> 2
- net RESET: track 0.00 -> 16.6 mm
- net MOSI: track 4.36 -> 11.1 mm
- net N$7: track 0.00 -> 6.05 mm
- net SCK: track 0.00 -> 4.52 mm
- net MISO: track 4.87 -> 9.12 mm
- net L-IN: track 159.5 -> 155.7 mm
- net N$2: track 7.20 -> 10.9 mm
- added copper zone on layer 1, net GND

Commit message: v0.5
Parts:
- moved C4 29.5 mm to (80.0, 42.3), turned to 90 degrees
- moved C1 14.9 mm to (68.2, 44.7)
- moved Q3 6.17 mm to (53.9, 10.8), turned to 0 degrees
- moved C2 5.14 mm to (80.1, 36.3)
- moved IC3 4.13 mm to (79.3, 28.5)
- moved IC1 3.49 mm to (70.2, 36.6)
- moved JP1 1.91 mm to (61.9, 38.6)
Routing:
- net +5V: track 100.4 -> 139.6 mm
- net N$11: track 3.79 -> 11.3 mm
- net RESET: track 16.6 -> 9.41 mm
- net LOAD: track 9.04 -> 15.4 mm
- net L-IN: track 155.7 -> 161.3 mm
- net MOSI: track 11.1 -> 6.56 mm
- net SCK: track 4.52 -> 0.00 mm
- net N-IN: track 151.6 -> 147.5 mm
- net OUT1: track 41.3 -> 45.4 mm, vias 2 -> 0
- net MISO: track 9.12 -> 5.08 mm
- net N$13: track 10.5 -> 7.72 mm
- net N$2: track 10.9 -> 13.1 mm
- net N$7: track 6.05 -> 4.38 mm

Commit message: v1.0
Parts:
- removed D1: DIODE1N4007, MyLib:SMA-DIODE
- removed JP1: (no value), pinhead:1X06
- added C5: 0.1, rcl:C0805
- added D2: 1N4446, diode:DO35-10
- added JP2, JP3: (no value), pinhead:1X02
- added JP4: (no value), pinhead:1X05
- added R1: 10k, rcl:R0805
- added U$1, U$2, U$3: MOUNTINGHOLE3.0THIN, MyLib:MOUNTINGHOLE_3.0_PLATEDTHIN
- C6: device rcl:153CLV-0605 -> rcl:E5-5
- Q3: value (none) -> BSS138
- moved R6 13.4 mm to (59.7, 19.5)
- moved C1 12.6 mm to (57.6, 37.9), turned to 90 degrees
- moved C4 6.01 mm to (80.9, 36.4), turned to 0 degrees
- moved C6 4.81 mm to (40.3, 22.7), turned to 270 degrees
- moved IC1 4.72 mm to (70.6, 41.3)
- moved Q3 3.36 mm to (54.2, 14.2), turned to 90 degrees
- moved C2 3.10 mm to (80.9, 33.3), turned to 0 degrees
- moved IC3 0.54 mm to (79.3, 27.9)
Connections:
- new net N$1: JP2.1, MD1.RX
- new net N$3: JP2.2, MD1.TX
- net +5V: now also D2.C, JP4.2, R1.1; no longer D1.C, JP1.1
- net GND: now also C5.2, JP3.1, JP4.1; no longer JP1.6
- net LOAD: now also IC1.2; no longer IC1.3
- net MISO: now also JP4.4; no longer JP1.3, MD1.TX
- net MOSI: now also JP4.5; no longer JP1.4, MD1.RX
- net N$13: now also D2.A; no longer D1.A
- net OUT1: now also IC1.3; no longer IC1.2
- net RESET: now also C5.1, JP3.2, R1.2; no longer JP1.5
- net SCK: now also JP4.3; no longer JP1.2
Routing:
- net +5V: track 139.6 -> 160.3 mm
- net N$1: track 0.00 -> 19.7 mm
- net N$3: track 0.00 -> 16.1 mm
- net GND: track 20.8 -> 7.78 mm
- net OUT1: track 45.4 -> 32.5 mm
- net LOAD: track 15.4 -> 22.6 mm
- net SCK: track 0.00 -> 5.47 mm
- net L-IN: track 161.3 -> 157.0 mm
- net RESET: track 9.41 -> 12.4 mm
- net N$7: track 4.38 -> 2.82 mm
- net N$11: track 11.3 -> 9.83 mm
- net MOSI: track 6.56 -> 5.50 mm
- net N$13: track 7.72 -> 8.72 mm
- net N$2: track 13.1 -> 12.6 mm
Other:
- board size 160 x 100 mm -> 93.5 x 51.5 mm
