File: L240-1.brd (EAGLE design)
At the start: 93.5 x 51.5 mm, 23 parts, among them IC1 TINY13-20SSU, IC3 ACS712-LC, K1 G2R2, Q3 BSS138, X4 MKDSN1,5/4-5,08

Commit message: v1.1
Parts:
- moved R1 2.23 mm to (74.2, 33.5)
- moved C1 2.00 mm to (57.6, 35.9), turned to 270 degrees
- moved R6 1.34 mm to (59.6, 18.2)
- moved C5 0.91 mm to (76.5, 43.2)
- moved JP2 0.32 mm to (57.3, 43.4)
Routing:
- net OUT1: track 32.5 -> 36.5 mm
- net RESET: track 12.4 -> 15.5 mm
- net N$2: track 12.6 -> 11.1 mm
- net N$11: track 9.83 -> 8.43 mm
- net +5V: track 160.3 -> 161.6 mm
- net L-IN: track 157.0 -> 156.5 mm
