File: L240-1.sch (EAGLE design)
At the start: 13 parts, among them IC1 TINY13-20SSU, IC2 LM1117IMPX-3.3, X2 22-23-2021, X3 MKDSN1,5/6-5,08

Commit message: relay
Parts:
- removed D9: DIODE1N4007, MyLib:DIODE1N4007
- added D1: DIODE1N4007, MyLib:DIODE1N4007
- added K1: G6RW, relay:G6RW
- added X1: MKDSN1,5/2-5,08, con-phoenix-508:MKDSN1,5/2-5,08
- X3: value MKDSN1,5/6-5,08 -> MKDSN1,5/2-5,08; device con-phoenix-508:MKDSN1,5/6-5,08 -> con-phoenix-508:MKDSN1,5/2-5,08
Connections:
- removed net GND1: Q3.S
- new net N$1: X1-1.KL, X3-2.KL
- new net N$2: K12.S, X3-1.KL
- new net N$3: K12.P, X1-2.KL
- net +5V: now also D1.C, K11.2; no longer D9.C
- net GND: now also Q3.S
- net N$13: now also D1.A, K11.1; no longer D9.A, X3-5.KL
Changed lines of the file:
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@@
 <part name="IC1" library="atmel" library_urn="urn:adsk.eagle:library:105" deviceset="TINY13" device="SSU" package3d_urn="urn:adsk.eagle:package:4358/1" technology="-20"/>
 <part name="R6" library="rcl" deviceset="R-EU_" device="R0805" value="50"/>
-<part name="X3" library="con-phoenix-508" library_urn="urn:adsk.eagle:library:176" deviceset="MKDSN1,5/6-5,08" device="" package3d_urn="urn:adsk.eagle:package:9634/1"/>
-<part name="D9" library="MyLib" deviceset="DIODE" device="1N4007"/>
 <part name="Q3" library="MyLib" deviceset="MOSFET-N" device="WIDE"/>
-<part name="SUPPLY1" library="supply2" library_urn="urn:adsk.eagle:library:372" deviceset="GND1" device=""/>
 <part name="GND12" library="supply1" deviceset="GND" device=""/>
 <part name="C13" library="rcl" deviceset="C-EU" device="C0805" value="0.1"/>
@@
 <part name="+3V2" library="supply1" deviceset="+3V3" device=""/>
 <part name="GND3" library="supply1" deviceset="GND" device=""/>
-<part name="P+3" library="supply1" deviceset="+5V" device=""/>
 <part name="+3V3" library="supply1" deviceset="+3V3" device=""/>
+<part name="X1" library="con-phoenix-508" library_urn="urn:adsk.eagle:library:176" deviceset="MKDSN1,5/2-5,08" device="" package3d_urn="urn:adsk.eagle:package:9630/1"/>
+<part name="K1" library="relay" library_urn="urn:adsk.eagle:library:339" deviceset="G6RW" device="" package3d_urn="urn:adsk.eagle:package:24332/1"/>
+<part name="X3" library="con-phoenix-508" library_urn="urn:adsk.eagle:library:176" deviceset="MKDSN1,5/2-5,08" device="" package3d_urn="urn:adsk.eagle:package:9630/1"/>
+<part name="P+1" library="supply1" deviceset="+5V" device=""/>
+<part name="D1" library="MyLib" deviceset="DIODE" device="1N4007"/>
+<part name="GND4" library="supply1" deviceset="GND" device=""/>
 </parts>
 <sheets>
@@
 <attribute name="VALUE" x="54.61" y="23.622" size="1.778" layer="96" rot="R180"/>
 </instance>
-<instance part="X3" gate="-5" x="91.44" y="27.94" smashed="yes">
-<attribute name="NAME" x="94.488" y="27.051" size="1.778" layer="95"/>
-</instance>
-<instance part="X3" gate="-6" x="91.44" y="38.1" smashed="yes">
-<attribute name="NAME" x="94.488" y="37.211" size="1.778" layer="95"/>
-</instance>
-<instance part="D9" gate="G$1" x="68.58" y="33.02" smashed="yes" rot="R90">
-<attribute name="NAME" x="66.548" y="30.48" size="1.778" layer="95" font="vector" rot="R90"/>
-<attribute name="VALUE" x="70.612" y="30.48" size="1.778" layer="96" font="vector" rot="R90" align="top-left"/>
-</instance>
 <instance part="Q3" gate="G$1" x="66.04" y="22.86" smashed="yes">
 <attribute name="NAME" x="71.12" y="23.495" size="1.27" layer="95"/>
 <attribute name="VALUE" x="71.12" y="21.59" size="1.27" layer="96"/>
 </instance>
-<instance part="SUPPLY1" gate="G$1" x="68.58" y="15.24" smashed="yes">
-<attribute name="VALUE" x="66.421" y="12.065" size="1.778" layer="96"/>
-</instance>
 <instance part="GND12" gate="1" x="43.18" y="99.06" smashed="yes">
 <attribute name="VALUE" x="40.64" y="96.52" size="1.778" layer="96"/>
@@
 <attribute name="VALUE" x="33.02" y="48.26" size="1.778" layer="96"/>
 </instance>
-<instance part="P+3" gate="1" x="68.58" y="43.18" smashed="yes">
-<attribute name="VALUE" x="66.04" y="38.1" size="1.778" layer="96" rot="R90"/>
-</instance>
 <instance part="+3V3" gate="G$1" x="20.32" y="119.38" smashed="yes">
 <attribute name="VALUE" x="17.78" y="114.3" size="1.778" layer="96" rot="R90"/>
+</instance>
+<instance part="X1" gate="-1" x="137.16" y="124.46" smashed="yes">
+<attribute name="NAME" x="140.208" y="123.571" size="1.778" layer="95"/>
+<attribute name="VALUE" x="134.62" y="120.777" size="1.778" layer="96"/>
+</instance>
+<instance part="X1" gate="-2" x="137.16" y="119.38" smashed="yes">
+<attribute name="NAME" x="140.208" y="118.491" size="1.778" layer="95"/>
+<attribute name="VALUE" x="134.62" y="115.697" size="1.778" layer="96"/>
+</instance>
+<instance part="K1" gate="1" x="96.52" y="142.24" smashed="yes" rot="R180">
+<attribute name="VALUE" x="95.25" y="139.319" size="1.778" layer="96" rot="R180"/>
+<attribute name="PART" x="95.25" y="137.16" size="1.778" layer="95" rot="R180"/>
+</instance>
+<instance part="K1" gate="2" x="114.3" y="142.24" smashed="yes">
+<attribute name="PART" x="116.84" y="142.24" size="1.778" layer="95"/>
+</instance>
+<instance part="X3" gate="-1" x="137.16" y="157.48" smashed="yes">
+<attribute name="NAME" x="140.208" y="156.591" size="1.778" layer="95"/>
+<attribute name="VALUE" x="134.62" y="153.797" size="1.778" layer="96"/>
+</instance>
+<instance part="X3" gate="-2" x="137.16" y="152.4" smashed="yes">
+<attribute name="NAME" x="140.208" y="151.511" size="1.778" layer="95"/>
+<attribute name="VALUE" x="134.62" y="148.717" size="1.778" layer="96"/>
+</instance>
+<instance part="P+1" gate="1" x="96.52" y="154.94" smashed="yes">
+<attribute name="VALUE" x="93.98" y="149.86" size="1.778" layer="96" rot="R90"/>
+</instance>
+<instance part="D1" gate="G$1" x="81.28" y="142.24" smashed="yes" rot="R90">
+<attribute name="NAME" x="79.248" y="139.7" size="1.778" layer="95" font="vector" rot="R90"/>
+<attribute name="VALUE" x="83.312" y="139.7" size="1.778" layer="96" font="vector" rot="R90" align="top-left"/>
+</instance>
+<instance part="GND4" gate="1" x="68.58" y="12.7" smashed="yes">
+<attribute name="VALUE" x="66.04" y="10.16" size="1.778" layer="96"/>
 </instance>
 </instances>
@@
 <net name="N$13" class="0">
 <segment>
-<pinref part="D9" gate="G$1" pin="A"/>
 <pinref part="Q3" gate="G$1" pin="D"/>
-<wire x1="68.58" y1="30.48" x2="68.58" y2="27.94" width="0.1524" layer="91"/>
-<wire x1="68.58" y1="27.94" x2="88.9" y2="27.94" width="0.1524" layer="91"/>
-<junction x="68.58" y="27.94"/>
-<pinref part="X3" gate="-5" pin="KL"/>
-</segment>
-</net>
-<net name="GND1" class="0">
-<segment>
-<pinref part="Q3" gate="G$1" pin="S"/>
-<pinref part="SUPPLY1" gate="G$1" pin="GND1"/>
+<wire x1="68.58" y1="27.94" x2="96.52" y2="27.94" width="0.1524" layer="91"/>
+<pinref part="D1" gate="G$1" pin="A"/>
+<wire x1="96.52" y1="134.62" x2="96.52" y2="27.94" width="0.1524" layer="91"/>
+<wire x1="81.28" y1="139.7" x2="81.28" y2="134.62" width="0.1524" layer="91"/>
+<wire x1="81.28" y1="134.62" x2="96.52" y2="134.62" width="0.1524" layer="91"/>
+<pinref part="K1" gate="1" pin="1"/>
+<wire x1="96.52" y1="134.62" x2="96.52" y2="137.16" width="0.1524" layer="91"/>
+<junction x="96.52" y="134.62"/>
 </segment>
 </net>
@@
 <wire x1="35.56" y1="60.96" x2="35.56" y2="53.34" width="0.1524" layer="91"/>
 </segment>
+<segment>
+<pinref part="GND4" gate="1" pin="GND"/>
+<pinref part="Q3" gate="G$1" pin="S"/>
+<wire x1="68.58" y1="15.24" x2="68.58" y2="17.78" width="0.1524" layer="91"/>
+</segment>
 </net>
 <net name="+5V" class="0">
@@
 </segment>
 <segment>
-<pinref part="D9" gate="G$1" pin="C"/>
-<pinref part="P+3" gate="1" pin="+5V"/>
-<wire x1="68.58" y1="35.56" x2="68.58" y2="40.64" width="0.1524" layer="91"/>
+<pinref part="K1" gate="1" pin="2"/>
+<pinref part="P+1" gate="1" pin="+5V"/>
+<wire x1="96.52" y1="147.32" x2="96.52" y2="149.86" width="0.1524" layer="91"/>
+<pinref part="D1" gate="G$1" pin="C"/>
+<wire x1="96.52" y1="149.86" x2="96.52" y2="152.4" width="0.1524" layer="91"/>
+<wire x1="96.52" y1="149.86" x2="81.28" y2="149.86" width="0.1524" layer="91"/>
+<wire x1="81.28" y1="149.86" x2="81.28" y2="144.78" width="0.1524" layer="91"/>
+<junction x="96.52" y="149.86"/>
 </segment>
 </net>
@@
 </segment>
 </net>
+<net name="N$1" class="0">
+<segment>
+<pinref part="X1" gate="-1" pin="KL"/>
+<pinref part="X3" gate="-2" pin="KL"/>
+<wire x1="134.62" y1="124.46" x2="134.62" y2="152.4" width="0.1524" layer="91"/>
+</segment>
+</net>
+<net name="N$2" class="0">
+<segment>
+<pinref part="X3" gate="-1" pin="KL"/>
+<pinref part="K1" gate="2" pin="S"/>
+<wire x1="134.62" y1="157.48" x2="109.22" y2="157.48" width="0.1524" layer="91"/>
+<wire x1="109.22" y1="157.48" x2="109.22" y2="147.32" width="0.1524" layer="91"/>
+</segment>
+</net>
+<net name="N$3" class="0">
+<segment>
+<pinref part="K1" gate="2" pin="P"/>
+<pinref part="X1" gate="-2" pin="KL"/>
+<wire x1="114.3" y1="139.7" x2="114.3" y2="119.38" width="0.1524" layer="91"/>
+<wire x1="114.3" y1="119.38" x2="134.62" y2="119.38" width="0.1524" layer="91"/>
+</segment>
+</net>

Commit message: wip
Parts:
- removed X1, X3: MKDSN1,5/2-5,08, con-phoenix-508:MKDSN1,5/2-5,08
- added C1, C3, C4: 0.1, rcl:C-EUC0805
- added C2: 1nF, rcl:C-EUC0805
- added IC3: ACS712-LC, allegro-2:ACS712-LC
- added U$1: KQ130, MyLib:KQ130
- added X4: MKDSN1,5/4-5,08, con-phoenix-508:MKDSN1,5/4-5,08
- K1: value G6RW -> G2R2; device relay:G6RW -> relay:G2R2
Connections:
- new net LOAD: IC1.PB3/PCINT3/CLKI/ADC3, IC3.VOUT
- new net N$4: IC3.IP-, IC3.IP-1, X4-1.KL
- new net N$6: K13.S, X4-2.KL
- new net N$7: C2.1, IC3.FILTER
- net +3V3: no longer IC1.VCC, JP1.2
- net +5V: now also C1.1, C3.1, C4.1, IC1.VCC, IC3.VCC, JP1.2; no longer IC2.IN
- net GND: now also C1.2, C2.2, C3.2, C4.2, IC3.GND
- net N$1: now also K12.S, X4-3.KL; no longer X1-1.KL, X3-2.KL
- net N$2: now also IC3.IP+, IC3.IP+1, K13.P; no longer K12.S, X3-1.KL
- net N$3: now also X4-4.KL; no longer X1-2.KL
Other:
- moved on the sheet: C13, C14, C15, D1, IC2, K1

Commit message: v0.1
Parts:
- removed C13, C14: 0.1, rcl:C-EUC0805
- removed C15: (no value), rcl:CPOL-EU153CLV-0605
- removed IC2: LM1117IMPX-3.3, lm1117:LM1117IMPX-3.3
- removed JP1: (no value), pinhead:PINHD-2X3
- removed U$1: KQ130, MyLib:KQ130
- removed X2: 22-23-2021, con-molex:22-23-2021
- added HLK1: HLK-PM013W, hi-link:HLK-PM013W
- added MD1: KQ130, MyLib:KQ130
Connections:
- net N$1 renamed N-OUT
- net N$6 renamed L-OUT
- removed net +3V3: C13.1, C14.1, C15.+, IC2.OUT, IC2.OUT1
- removed net N$3: K12.P, X4-4.KL
- removed net N$4: IC3.IP-, IC3.IP-1, X4-1.KL
- new net L-IN: HLK1.AC2, IC3.IP-, IC3.IP-1, MD1.AC2, X4-1.KL
- new net N-IN: HLK1.AC1, K12.P, MD1.AC1, X4-4.KL
- net +5V: now also HLK1.+VO, MD1.VCC@1, MD1.VCC@2; no longer JP1.2, X2-1.S
- net GND: now also HLK1.-VO, MD1.GND; no longer C13.2, C14.2, C15.-, IC2.GND, JP1.6, X2-2.S
- net MISO: now also MD1.TX; no longer JP1.1
- net MOSI: now also MD1.RX; no longer JP1.4
- net RESET: no longer JP1.5
- net SCK: no longer JP1.3

Commit message: v0.2
Connections:
- net +5V: now also K11.1; no longer K11.2
- net N$13: now also K11.2; no longer K11.1
Other:
- moved on the sheet: K1
Changed lines of the file:
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@@
 <attribute name="VALUE" x="66.04" y="10.16" size="1.778" layer="96"/>
 </instance>
-<instance part="K1" gate="1" x="106.68" y="38.1" smashed="yes" rot="R180">
-<attribute name="VALUE" x="105.41" y="35.179" size="1.778" layer="96" rot="R180"/>
-<attribute name="PART" x="105.41" y="33.02" size="1.778" layer="95" rot="R180"/>
+<instance part="K1" gate="1" x="106.68" y="38.1" smashed="yes">
+<attribute name="VALUE" x="107.95" y="41.021" size="1.778" layer="96"/>
+<attribute name="PART" x="107.95" y="43.18" size="1.778" layer="95"/>
 </instance>
 <instance part="K1" gate="2" x="124.46" y="5.08" smashed="yes">
@@
 <wire x1="96.52" y1="35.56" x2="96.52" y2="30.48" width="0.1524" layer="91"/>
 <wire x1="96.52" y1="30.48" x2="106.68" y2="30.48" width="0.1524" layer="91"/>
-<pinref part="K1" gate="1" pin="1"/>
+<pinref part="K1" gate="1" pin="2"/>
 <wire x1="106.68" y1="33.02" x2="106.68" y2="30.48" width="0.1524" layer="91"/>
 <junction x="106.68" y="30.48"/>
@@
 <wire x1="96.52" y1="40.64" x2="96.52" y2="45.72" width="0.1524" layer="91"/>
 <wire x1="96.52" y1="45.72" x2="106.68" y2="45.72" width="0.1524" layer="91"/>
-<pinref part="K1" gate="1" pin="2"/>
-<wire x1="106.68" y1="45.72" x2="106.68" y2="43.18" width="0.1524" layer="91"/>
+<pinref part="K1" gate="1" pin="1"/>
+<wire x1="106.68" y1="43.18" x2="106.68" y2="45.72" width="0.1524" layer="91"/>
 <junction x="106.68" y="45.72"/>
 </segment>

Commit message: v0.3
Connections:
- net LOAD: now also IC1.PB4/PCINT4/ADC2; no longer IC1.PB3/PCINT3/CLKI/ADC3
- net OUT1: now also IC1.PB3/PCINT3/CLKI/ADC3; no longer IC1.PB4/PCINT4/ADC2
Other:
- moved on the sheet: K1, X4-1, X4-2, X4-3, X4-4
Changed lines of the file:
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@@
 <attribute name="PART" x="107.95" y="43.18" size="1.778" layer="95"/>
 </instance>
-<instance part="K1" gate="2" x="124.46" y="5.08" smashed="yes">
-<attribute name="PART" x="127" y="5.08" size="1.778" layer="95"/>
-</instance>
-<instance part="K1" gate="3" x="134.62" y="101.6" smashed="yes">
-<attribute name="PART" x="137.16" y="101.6" size="1.778" layer="95"/>
+<instance part="K1" gate="2" x="182.88" y="22.86" smashed="yes">
+<attribute name="PART" x="185.42" y="22.86" size="1.778" layer="95"/>
+</instance>
+<instance part="K1" gate="3" x="134.62" y="134.62" smashed="yes">
+<attribute name="PART" x="137.16" y="134.62" size="1.778" layer="95"/>
 </instance>
 <instance part="IC3" gate="G$1" x="132.08" y="76.2" smashed="yes" rot="MR0">
@@
 <attribute name="VALUE" x="129.54" y="63.5" size="1.778" layer="96" rot="MR0"/>
 </instance>
-<instance part="X4" gate="-1" x="157.48" y="48.26" smashed="yes">
-<attribute name="NAME" x="160.528" y="47.371" size="1.778" layer="95"/>
-<attribute name="VALUE" x="154.94" y="44.577" size="1.778" layer="96"/>
-</instance>
-<instance part="X4" gate="-2" x="157.48" y="119.38" smashed="yes">
-<attribute name="NAME" x="160.528" y="118.491" size="1.778" layer="95"/>
-</instance>
-<instance part="X4" gate="-3" x="154.94" y="17.78" smashed="yes">
-<attribute name="NAME" x="157.988" y="16.891" size="1.778" layer="95"/>
-</instance>
-<instance part="X4" gate="-4" x="154.94" y="2.54" smashed="yes">
-<attribute name="NAME" x="157.988" y="1.651" size="1.778" layer="95"/>
+<instance part="X4" gate="-1" x="162.56" y="53.34" smashed="yes">
+<attribute name="NAME" x="165.608" y="52.451" size="1.778" layer="95"/>
+<attribute name="VALUE" x="160.02" y="49.657" size="1.778" layer="96"/>
+</instance>
+<instance part="X4" gate="-2" x="157.48" y="152.4" smashed="yes">
+<attribute name="NAME" x="160.528" y="151.511" size="1.778" layer="95"/>
+</instance>
+<instance part="X4" gate="-3" x="213.36" y="35.56" smashed="yes">
+<attribute name="NAME" x="216.408" y="34.671" size="1.778" layer="95"/>
+</instance>
+<instance part="X4" gate="-4" x="213.36" y="20.32" smashed="yes">
+<attribute name="NAME" x="216.408" y="19.431" size="1.778" layer="95"/>
 </instance>
 <instance part="P+3" gate="1" x="114.3" y="96.52" smashed="yes">
@@
 <pinref part="R6" gate="G$1" pin="2"/>
 <wire x1="45.72" y1="20.32" x2="30.48" y2="20.32" width="0.1524" layer="91"/>
-<pinref part="IC1" gate="G$1" pin="PB4/PCINT4/ADC2"/>
-<wire x1="38.1" y1="66.04" x2="30.48" y2="66.04" width="0.1524" layer="91"/>
-<wire x1="30.48" y1="66.04" x2="30.48" y2="20.32" width="0.1524" layer="91"/>
+<wire x1="30.48" y1="68.58" x2="30.48" y2="20.32" width="0.1524" layer="91"/>
+<label x="30.48" y="38.1" size="1.778" layer="95"/>
+<pinref part="IC1" gate="G$1" pin="PB3/PCINT3/CLKI/ADC3"/>
+<wire x1="30.48" y1="68.58" x2="38.1" y2="68.58" width="0.1524" layer="91"/>
 </segment>
 </net>
@@
 <wire x1="96.52" y1="35.56" x2="96.52" y2="30.48" width="0.1524" layer="91"/>
 <wire x1="96.52" y1="30.48" x2="106.68" y2="30.48" width="0.1524" layer="91"/>
+<junction x="106.68" y="30.48"/>
 <pinref part="K1" gate="1" pin="2"/>
 <wire x1="106.68" y1="33.02" x2="106.68" y2="30.48" width="0.1524" layer="91"/>
-<junction x="106.68" y="30.48"/>
 </segment>
 </net>
@@
 <net name="N-IN" class="0">
 <segment>
-<pinref part="X4" gate="-4" pin="KL"/>
-<wire x1="124.46" y1="2.54" x2="152.4" y2="2.54" width="0.1524" layer="91"/>
-<pinref part="K1" gate="2" pin="P"/>
-<label x="139.7" y="2.54" size="1.778" layer="95"/>
-</segment>
-<segment>
 <pinref part="MD1" gate="G$1" pin="AC1"/>
 <wire x1="-43.18" y1="63.5" x2="-86.36" y2="63.5" width="0.1524" layer="91"/>
@@
 <wire x1="-81.28" y1="96.52" x2="-101.6" y2="96.52" width="0.1524" layer="91"/>
 </segment>
+<segment>
+<pinref part="K1" gate="2" pin="P"/>
+<wire x1="149.86" y1="20.32" x2="182.88" y2="20.32" width="0.1524" layer="91"/>
+<pinref part="X4" gate="-4" pin="KL"/>
+<wire x1="182.88" y1="20.32" x2="210.82" y2="20.32" width="0.1524" layer="91"/>
+<label x="195.58" y="20.32" size="1.778" layer="95"/>
+</segment>
 </net>
 <net name="N-OUT" class="0">
@@
 <pinref part="K1" gate="2" pin="S"/>
 <pinref part="X4" gate="-3" pin="KL"/>
-<wire x1="119.38" y1="10.16" x2="119.38" y2="17.78" width="0.1524" layer="91"/>
-<wire x1="119.38" y1="17.78" x2="152.4" y2="17.78" width="0.1524" layer="91"/>
-<label x="139.7" y="17.78" size="1.778" layer="95"/>
+<wire x1="177.8" y1="27.94" x2="177.8" y2="35.56" width="0.1524" layer="91"/>
+<wire x1="177.8" y1="35.56" x2="210.82" y2="35.56" width="0.1524" layer="91"/>
+<label x="198.12" y="35.56" size="1.778" layer="95"/>
 </segment>
 </net>
@@
 <segment>
 <pinref part="K1" gate="3" pin="S"/>
-<wire x1="127" y1="106.68" x2="129.54" y2="106.68" width="0.1524" layer="91"/>
+<wire x1="127" y1="139.7" x2="129.54" y2="139.7" width="0.1524" layer="91"/>
 <pinref part="X4" gate="-2" pin="KL"/>
-<wire x1="127" y1="106.68" x2="127" y2="119.38" width="0.1524" layer="91"/>
-<wire x1="127" y1="119.38" x2="154.94" y2="119.38" width="0.1524" layer="91"/>
-<label x="137.16" y="119.38" size="1.778" layer="95"/>
-</segment>
-</net>
-<net name="N$2" class="0">
-<segment>
-<pinref part="K1" gate="3" pin="P"/>
-<pinref part="IC3" gate="G$1" pin="IP+1"/>
-<wire x1="134.62" y1="99.06" x2="134.62" y2="91.44" width="0.1524" layer="91"/>
-<pinref part="IC3" gate="G$1" pin="IP+"/>
-<wire x1="134.62" y1="91.44" x2="139.7" y2="91.44" width="0.1524" layer="91"/>
-<junction x="134.62" y="91.44"/>
+<wire x1="127" y1="139.7" x2="127" y2="152.4" width="0.1524" layer="91"/>
+<wire x1="127" y1="152.4" x2="154.94" y2="152.4" width="0.1524" layer="91"/>
+<label x="137.16" y="152.4" size="1.778" layer="95"/>
 </segment>
 </net>
 <net name="L-IN" class="0">
-<segment>
-<pinref part="IC3" gate="G$1" pin="IP-"/>
-<pinref part="IC3" gate="G$1" pin="IP-1"/>
-<wire x1="139.7" y1="60.96" x2="134.62" y2="60.96" width="0.1524" layer="91"/>
-<wire x1="134.62" y1="60.96" x2="134.62" y2="48.26" width="0.1524" layer="91"/>
-<junction x="134.62" y="60.96"/>
-<pinref part="X4" gate="-1" pin="KL"/>
-<wire x1="134.62" y1="48.26" x2="154.94" y2="48.26" width="0.1524" layer="91"/>
-<label x="142.24" y="48.26" size="1.778" layer="95"/>
-</segment>
 <segment>
 <pinref part="MD1" gate="G$1" pin="AC2"/>
@@
 <label x="-96.52" y="101.6" size="1.778" layer="95"/>
 </segment>
+<segment>
+<wire x1="139.7" y1="53.34" x2="160.02" y2="53.34" width="0.1524" layer="91"/>
+<pinref part="X4" gate="-1" pin="KL"/>
+<label x="149.86" y="53.34" size="1.778" layer="95"/>
+<pinref part="IC3" gate="G$1" pin="IP-"/>
+<pinref part="IC3" gate="G$1" pin="IP-1"/>
+<wire x1="134.62" y1="60.96" x2="139.7" y2="60.96" width="0.1524" layer="91"/>
+<wire x1="139.7" y1="53.34" x2="139.7" y2="60.96" width="0.1524" layer="91"/>
+<junction x="139.7" y="60.96"/>
+</segment>
 </net>
 <net name="LOAD" class="0">
 <segment>
-<pinref part="IC1" gate="G$1" pin="PB3/PCINT3/CLKI/ADC3"/>
-<wire x1="38.1" y1="68.58" x2="27.94" y2="68.58" width="0.1524" layer="91"/>
-<wire x1="27.94" y1="68.58" x2="27.94" y2="45.72" width="0.1524" layer="91"/>
+<wire x1="27.94" y1="66.04" x2="27.94" y2="45.72" width="0.1524" layer="91"/>
 <wire x1="27.94" y1="45.72" x2="88.9" y2="45.72" width="0.1524" layer="91"/>
 <wire x1="88.9" y1="45.72" x2="88.9" y2="78.74" width="0.1524" layer="91"/>
@@
 <wire x1="88.9" y1="78.74" x2="116.84" y2="78.74" width="0.1524" layer="91"/>
 <label x="68.58" y="45.72" size="1.778" layer="95"/>
+<pinref part="IC1" gate="G$1" pin="PB4/PCINT4/ADC2"/>
+<wire x1="38.1" y1="66.04" x2="27.94" y2="66.04" width="0.1524" layer="91"/>
 </segment>
 </net>
@@
 </segment>
 </net>
+<net name="N$2" class="0">
+<segment>
+<pinref part="IC3" gate="G$1" pin="IP+"/>
+<pinref part="IC3" gate="G$1" pin="IP+1"/>
+<wire x1="134.62" y1="91.44" x2="139.7" y2="91.44" width="0.1524" layer="91"/>
+<pinref part="K1" gate="3" pin="P"/>
+<wire x1="134.62" y1="91.44" x2="134.62" y2="132.08" width="0.1524" layer="91"/>
+<junction x="134.62" y="91.44"/>
+</segment>
+</net>
