File: L240-1.sch (EAGLE design)
At the start: 15 parts, among them IC1 TINY13-20SSU, IC3 ACS712-LC, K1 G2R2, X4 MKDSN1,5/4-5,08

Commit message: v0.4
Parts:
- added JP1: (no value), pinhead:PINHD-1X6
Connections:
- net +5V: now also JP1.1
- net GND: now also JP1.6
- net MISO: now also JP1.3
- net MOSI: now also JP1.4
- net RESET: now also JP1.5
- net SCK: now also JP1.2
Changed lines of the file:
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@@
 <part name="GND2" library="supply1" deviceset="GND" device=""/>
 <part name="P+6" library="supply1" deviceset="+5V" device=""/>
+<part name="JP1" library="pinhead" library_urn="urn:adsk.eagle:library:325" deviceset="PINHD-1X6" device="" package3d_urn="urn:adsk.eagle:package:22472/2"/>
 </parts>
 <sheets>
@@
 <attribute name="VALUE" x="-1.016" y="99.441" size="1.778" layer="96"/>
 </instance>
-<instance part="GND22" gate="1" x="-7.62" y="25.4" smashed="yes">
-<attribute name="VALUE" x="-10.16" y="22.86" size="1.778" layer="96"/>
+<instance part="GND22" gate="1" x="2.54" y="-5.08" smashed="yes">
+<attribute name="VALUE" x="0" y="-7.62" size="1.778" layer="96"/>
 </instance>
 <instance part="GND3" gate="1" x="35.56" y="50.8" smashed="yes">
@@
 <attribute name="VALUE" x="33.02" y="83.82" size="1.778" layer="96" rot="R90"/>
 </instance>
-<instance part="P+5" gate="1" x="-7.62" y="45.72" smashed="yes">
-<attribute name="VALUE" x="-10.16" y="40.64" size="1.778" layer="96" rot="R90"/>
+<instance part="P+5" gate="1" x="2.54" y="20.32" smashed="yes">
+<attribute name="VALUE" x="0" y="15.24" size="1.778" layer="96" rot="R90"/>
 </instance>
 <instance part="C3" gate="G$1" x="7.62" y="104.14" smashed="yes">
@@
 <instance part="P+6" gate="1" x="-10.16" y="66.04" smashed="yes">
 <attribute name="VALUE" x="-12.7" y="60.96" size="1.778" layer="96" rot="R90"/>
+</instance>
+<instance part="JP1" gate="A" x="12.7" y="5.08" smashed="yes">
+<attribute name="NAME" x="6.35" y="15.875" size="1.778" layer="95"/>
+<attribute name="VALUE" x="6.35" y="-5.08" size="1.778" layer="96"/>
 </instance>
 </instances>
@@
 </segment>
 <segment>
-<pinref part="GND22" gate="1" pin="GND"/>
-<wire x1="-15.24" y1="30.48" x2="-7.62" y2="30.48" width="0.1524" layer="91"/>
-<wire x1="-7.62" y1="30.48" x2="-7.62" y2="27.94" width="0.1524" layer="91"/>
-</segment>
-<segment>
 <pinref part="IC1" gate="G$1" pin="GND"/>
 <wire x1="38.1" y1="60.96" x2="35.56" y2="60.96" width="0.1524" layer="91"/>
@@
 <pinref part="GND2" gate="1" pin="GND"/>
 <wire x1="-17.78" y1="81.28" x2="-12.7" y2="81.28" width="0.1524" layer="91"/>
+</segment>
+<segment>
+<pinref part="GND22" gate="1" pin="GND"/>
+<pinref part="JP1" gate="A" pin="6"/>
+<wire x1="2.54" y1="-2.54" x2="2.54" y2="0" width="0.1524" layer="91"/>
+<wire x1="2.54" y1="0" x2="10.16" y2="0" width="0.1524" layer="91"/>
 </segment>
 </net>
@@
 </segment>
 <segment>
-<wire x1="-15.24" y1="35.56" x2="-7.62" y2="35.56" width="0.1524" layer="91"/>
-<wire x1="-7.62" y1="35.56" x2="-7.62" y2="43.18" width="0.1524" layer="91"/>
-<pinref part="P+5" gate="1" pin="+5V"/>
-</segment>
-<segment>
 <pinref part="MD1" gate="G$1" pin="VCC@2"/>
 <pinref part="MD1" gate="G$1" pin="VCC@1"/>
@@
 <wire x1="-10.16" y1="60.96" x2="-10.16" y2="63.5" width="0.1524" layer="91"/>
 </segment>
+<segment>
+<pinref part="P+5" gate="1" pin="+5V"/>
+<pinref part="JP1" gate="A" pin="1"/>
+<wire x1="2.54" y1="17.78" x2="2.54" y2="12.7" width="0.1524" layer="91"/>
+<wire x1="2.54" y1="12.7" x2="10.16" y2="12.7" width="0.1524" layer="91"/>
+</segment>
 </net>
 <net name="MOSI" class="0">
 <segment>
-<wire x1="-15.24" y1="33.02" x2="0" y2="33.02" width="0.1524" layer="91"/>
-<label x="-5.08" y="33.02" size="1.778" layer="95"/>
+<wire x1="-5.08" y1="5.08" x2="10.16" y2="5.08" width="0.1524" layer="91"/>
+<label x="-2.54" y="5.08" size="1.778" layer="95"/>
+<pinref part="JP1" gate="A" pin="4"/>
 </segment>
 <segment>
@@
 <net name="MISO" class="0">
 <segment>
-<wire x1="-22.86" y1="35.56" x2="-35.56" y2="35.56" width="0.1524" layer="91"/>
-<label x="-35.56" y="35.56" size="1.778" layer="95"/>
+<wire x1="10.16" y1="7.62" x2="-2.54" y2="7.62" width="0.1524" layer="91"/>
+<label x="-2.54" y="7.62" size="1.778" layer="95"/>
+<pinref part="JP1" gate="A" pin="3"/>
 </segment>
 <segment>
@@
 <net name="SCK" class="0">
 <segment>
-<wire x1="-22.86" y1="33.02" x2="-35.56" y2="33.02" width="0.1524" layer="91"/>
-<label x="-35.56" y="33.02" size="1.778" layer="95"/>
+<wire x1="10.16" y1="10.16" x2="-2.54" y2="10.16" width="0.1524" layer="91"/>
+<label x="-2.54" y="10.16" size="1.778" layer="95"/>
+<pinref part="JP1" gate="A" pin="2"/>
 </segment>
 <segment>
@@
 <net name="RESET" class="0">
 <segment>
-<wire x1="-22.86" y1="30.48" x2="-35.56" y2="30.48" width="0.1524" layer="91"/>
-<label x="-35.56" y="30.48" size="1.778" layer="95"/>
-</segment>
-<segment>
+<wire x1="10.16" y1="2.54" x2="-2.54" y2="2.54" width="0.1524" layer="91"/>
+<label x="-2.54" y="2.54" size="1.778" layer="95"/>
+<pinref part="JP1" gate="A" pin="5"/>
+</segment>
+<segment>

Commit message: v1.0
Parts:
- removed D1: DIODE1N4007, MyLib:DIODE1N4007
- removed JP1: (no value), pinhead:PINHD-1X6
- added C5: 0.1, rcl:C-EUC0805
- added D2: 1N4446, diode:1N4446
- added JP2, JP3: (no value), pinhead:PINHD-1X2
- added JP4: (no value), pinhead:PINHD-1X5
- added R1: 10k, rcl:R-EU_R0805
- added U$1, U$2, U$3: MOUNTINGHOLE3.0THIN, MyLib:MOUNTINGHOLE3.0THIN
- C6: device rcl:CPOL-EU153CLV-0605 -> rcl:CPOL-EUE5-5
- Q3: value (none) -> BSS138
Connections:
- new net N$1: JP2.1, MD1.RX
- new net N$3: JP2.2, MD1.TX
- net +5V: now also D2.C, JP4.2, R1.1; no longer D1.C, JP1.1
- net GND: now also C5.2, JP3.1, JP4.1; no longer JP1.6
- net LOAD: now also IC1.PB3/PCINT3/CLKI/ADC3; no longer IC1.PB4/PCINT4/ADC2
- net MISO: now also JP4.4; no longer JP1.3, MD1.TX
- net MOSI: now also JP4.5; no longer JP1.4, MD1.RX
- net N$13: now also D2.A; no longer D1.A
- net OUT1: now also IC1.PB4/PCINT4/ADC2; no longer IC1.PB3/PCINT3/CLKI/ADC3
- net RESET: now also C5.1, JP3.2, R1.2; no longer JP1.5
- net SCK: now also JP4.3; no longer JP1.2
Other:
- moved on the sheet: C6, MD1

Commit message: v1.1
Other:
- moved on the sheet: C1, C10, C3, C4, C5, C6, HLK1, JP2, JP3, K1, MD1, R1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
